Commit message: snapshot of the repo on CARIS computer on Feb 3 2023, adding gantry to model and modification for Maram's AR learning experiment

File: iiwa_description/urdf/iiwa14.urdf.xacro (robot description, xacro)
@@ -1,17 +1,58 @@
 <?xml version="1.0"?>
-<robot name="iiwa14" xmlns:xacro="http://www.ros.org/wiki/xacro">
+<!-- Here we define the robot, we named it "iiwa14_tool" -->
+<robot xmlns:xacro="http://www.ros.org/wiki/xacro" name="iiwa14">
   <!-- Import Rviz colors -->
   <xacro:include filename="$(find iiwa_description)/urdf/materials.xacro" />
-  <!--Import the lbr iiwa macro -->
+  <!--Import the iiwa14 macro -->
   <xacro:include filename="$(find iiwa_description)/urdf/iiwa14.xacro"/>
+  <!--Import the gantry urdf-->
+  <xacro:include filename="$(find gantry3)/urdf/gantry3.urdf" />
+  <!--  Arguments for the iiwa14 macro  -->
   <xacro:arg name="hardware_interface" default="PositionJointInterface"/>
   <xacro:arg name="robot_name" default="iiwa"/>
-  <xacro:arg name="origin_xyz" default="0 0 0"/>
-  <xacro:arg name="origin_rpy" default="0 0 0"/>
-  <!-- Fix to world just for testing -->
-  <link name="world"/>
-  <!--iiwa-->
+  <link name="world" />
+  <!-- Here we insert an iiwa14 robot in the scene, it's origin is just on top of the box previously defined. You can use 0,0,0 if you don't have that. -->
   <xacro:iiwa14 hardware_interface="$(arg hardware_interface)" robot_name="$(arg robot_name)" parent="world">
-    <origin xyz="$(arg origin_xyz)" rpy="$(arg origin_rpy)" />
+    <origin xyz="-0.2 0 1.985" rpy="${radians(0)} ${radians(180)} 0"/>
   </xacro:iiwa14>
+  <!-- Tool properties -->
+  <property name="tool_mass" value="0.200" />
+  <property name="tool_joint_offset" value="0.00 0.00 0.08" />
+  <!-- Change the offset for end effector origin -->
+  <property name="tool_link_offset" value="-0.075 0.00 0" />
+  <!--  Here we define a dummy joint between the tip of the iiwa14 and the base of the tool.
+  There is no offset between the two, that means the tool is attached at the robot flange. -->
+  <joint name="tool_joint" type="fixed">
+    <parent link="iiwa_link_ee" />
+    <child link = "tool_link" />
+    <origin xyz="${tool_joint_offset}" rpy="0 ${PI/2.0} 0" />
+  </joint>
+  <!-- Here we define the geometry of the tool. We designed the tool ourselves, so we have a mesh file that represents it.
+  Else, one can define it using a geometric representation that approximate it, like a cylinder (see commented lines) -->
+  <link name="tool_link">
+    <visual>
+      <origin xyz="0 0 0" rpy="0 ${PI/2.0} 0"/>
+      <geometry>
+	<!-- <mesh filename="package://iiwa_tool_description/meshes/visual/tool.stl"/> -->
+	<cylinder length="0.16" radius="0.01"/>
+      </geometry>
+      <material name="Grey"/>
+    </visual>
+    <collision>
+      <origin xyz="0 0 0" rpy="0 ${PI/2.0} 0"/>
+      <geometry>
+	<!-- <mesh filename="package://iiwa_tool_description/meshes/visual/tool.stl"/> -->
+	<cylinder length="0.17" radius="0.025"/>
+      </geometry>
+      <material name="Grey"/>
+    </collision>
+  </link>
+  <!--  Here we define another dummy joint. It is placed at the end of the tool, so we can then attach a frame at its TCP for control -->
+  <joint name="tool_tip_joint" type="fixed">
+    <parent link="tool_link" />
+    <child link = "tool_link_ee" />
+    <origin xyz="${tool_link_offset}" rpy="0 0 0" />
+  </joint>
+  <!--  ohThe TCP frame is here defined -->
+  <link name="tool_link_ee"/>
 </robot>
